File: HARDWARE/Embedded-Board/Embedded-Board.kicad_sch (KiCad schematic)
At the start: 5 parts, among them J1 SENSOR SOCKET, J2 POWER-pins, J3 Conn_02x20_Odd_Even, SW1 SW_Push, SW2 RotaryEncoder_Switch

Commit message: Schematic v1 done
Other:
- company: (none) -> Drawn by Nicolas Viale
- title: (none) -> Low Cost VIS/NIF Spectrometer
Changed lines of the file:
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@@
 	(paper "A4")
 	(title_block
+		(title "Low Cost VIS/NIF Spectrometer")
 		(date "2025-04-08")
+		(rev "v1")
+		(company "Drawn by Nicolas Viale")
 	)
 	(rectangle
