File: HARDWARE/Embedded-Board/RP2040.kicad_sch (KiCad schematic)
At the start: 23 parts, among them J9 DEBUG, SW5 BOOT, U2 W25Q16JVS, U3 RP2040, Y1 12MHz

Commit message: Schematic v1 done
Connections:
- net E-PAPER-DC: now reaches U3.11 (GPIO8)
- net E-PAPER-CS: now reaches U3.12 (GPIO9)
- net E-PAPER-SCK: now reaches U3.13 (GPIO10)
- net E-PAPER-MOSI: now reaches U3.14 (GPIO11)
- net E-PAPER-RST: now reaches U3.15 (GPIO12)
- net E-PAPER-BUSY: now reaches U3.16 (GPIO13)
- net PUSH-SWITCH: now reaches U3.18 (GPIO15)
- net SENSOR-SDA: now reaches U3.2 (GPIO0)
- net SENSOR-SCL: now reaches U3.3 (GPIO1)
- net ENC-A: now reaches U3.5 (GPIO3)
- net ENC-PSH: now reaches U3.6 (GPIO4)
- net ENC-B: now reaches U3.7 (GPIO5)
- no-connect marks 0 -> 18
Other:
- company: (none) -> Drawn by Nicoals Viale
- title: (none) -> Low Cost VIS/NIF Spectrometer
