File: HARDWARE/Embedded-Board/RP2040.kicad_sch (KiCad schematic)
At the start: 23 parts, among them J9 DEBUG, SW5 BOOT, U2 W25Q16JVS, U3 RP2040, Y1 12MHz

Commit message: New PCB design for JLCPCB
Parts:
- removed J9: DEBUG, Connector_PinSocket_2.54mm:PinSocket_1x02_P2.54mm_Vertical, symbol Connector:Conn_01x02_Socket
- added J6: GPIO PINS, Connector_PinHeader_2.54mm:PinHeader_1x09_P2.54mm_Vertical, symbol Connector:Conn_01x09_Pin
- added TP6: SWCLK, TestPoint:TestPoint_Pad_D1.0mm, symbol Connector:TestPoint
- added TP7: SWD, TestPoint:TestPoint_Pad_D1.0mm, symbol Connector:TestPoint
Connections:
- net GND: now also J6.1 (Pin_1)
- net at U3.25 (SWD): now also TP7.1
- net at U3.24 (SWCLK): now also TP6.1
- net at U3.27 (GPIO16): now also J6.2 (Pin_2)
- net at U3.28 (GPIO17): now also J6.3 (Pin_3)
- net at U3.29 (GPIO18): now also J6.4 (Pin_4)
- net at U3.30 (GPIO19): now also J6.5 (Pin_5)
- net at U3.31 (GPIO20): now also J6.6 (Pin_6)
- net at U3.32 (GPIO21): now also J6.7 (Pin_7)
- net at U3.38 (GPIO26_ADC0): now also J6.8 (Pin_8)
- net at U3.39 (GPIO27_ADC1): now also J6.9 (Pin_9)
- no-connect marks 16 -> 8
Other:
- title: Low Cost VIS/NIF Spectrometer -> Low Cost VIS/NIR Spectrometer

Commit message: Final PCB version
Connections:
- net SENSOR-INT: now also U3.8 (GPIO6); no longer U3.36 (GPIO24)
- net SENSOR-RST: now also U3.9 (GPIO7); no longer U3.37 (GPIO25)
