File: HARDWARE/Embedded-Board/POWER.kicad_sch (KiCad schematic)
At the start: 36 parts, among them J11 USB_C_Receptacle_USB2.0, Q1 MMUN2133LT1G, SW3 SW_Push_SPDT, U1 MCP73831-2-OT, U18 LM1117-3.3, U4 TPS61090

Commit message: Schematic v1 done
Other:
- company: (none) -> Drawn by Nicolas Viale
- title: (none) -> Low Cost VIS/NIF Spectrometer
Changed lines of the file:
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@@
 	(generator_version "9.0")
 	(paper "A4")
+	(title_block
+		(title "Low Cost VIS/NIF Spectrometer")
+		(date "2025-04-08")
+		(rev "v1")
+		(company "Drawn by Nicolas Viale")
+	)
 	(rectangle
 		(start 15.24 81.28)

Commit message: New PCB design for JLCPCB
Parts:
- C6: footprint Capacitor_SMD:CP_Elec_6.3x7.7 -> Capacitor_SMD:C_0805_2012Metric
Other:
- title: Low Cost VIS/NIF Spectrometer -> Low Cost VIS/NIR Spectrometer
Changed lines of the file:
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@@
 	(paper "A4")
 	(title_block
-		(title "Low Cost VIS/NIF Spectrometer")
+		(title "Low Cost VIS/NIR Spectrometer")
 		(date "2025-04-08")
 		(rev "v1")
@@
 			)
 		)
-		(property "Footprint" "Capacitor_SMD:CP_Elec_6.3x7.7"
+		(property "Footprint" "Capacitor_SMD:C_0805_2012Metric"
 			(at 266.3952 38.1 0)
 			(effects

Commit message: Final PCB version
Parts:
- added JP1: VBUS-5V, Jumper:SolderJumper-2_P1.3mm_Open_TrianglePad1.0x1.5mm, symbol Jumper:SolderJumper_2_Open
- added JP2: OUT-5V, Jumper:SolderJumper-2_P1.3mm_Bridged_Pad1.0x1.5mm, symbol Jumper:SolderJumper_2_Bridged
- C2, C3, C5: footprint Capacitor_SMD:C_0603_1608Metric -> Capacitor_SMD:C_0805_2012Metric
- C6: footprint Capacitor_SMD:C_0805_2012Metric -> Capacitor_SMD:C_1206_3216Metric
Connections:
- net +5V: now also JP1.2 (B), JP2.2 (B); no longer R18.2, U4.1 (VOUT), U4.15 (VOUT), U4.16 (VOUT)
- net VBUS: now also JP1.1 (A)
- new net: JP2.1 (A), R18.2, U4.1 (VOUT), U4.15 (VOUT), U4.16 (VOUT)
